File: pcb/LEDGrid.kicad_sch (KiCad schematic)
At the start: 0 parts

Commit message: updates
Other:
- removed sheet LED Row25
- removed sheet LED Row26
- removed sheet LED Row27
- removed sheet LED Row28
- removed sheet LED Row29
- removed sheet LED Row30
- removed sheet LED Row31
- removed sheet LED Row32
- removed sheet LED Row33
- removed sheet LED Row34
- removed sheet LED Row35
- removed sheet LED Row36
- removed sheet LED Row37
- removed sheet LED Row38
- removed sheet LED Row39
- removed sheet LED Row40
- removed sheet LED Row41
- removed sheet LED Row42
- removed sheet LED Row43
- removed sheet LED Row44
- removed sheet LED Row45
- removed sheet LED Row46
- removed sheet LED Row47
- removed sheet LED Row48
- removed sheet LED Row49
- removed sheet LED Row50
- removed sheet LED Row51
- removed sheet LED Row52
- removed sheet LED Row53
- removed sheet LED Row54
- removed sheet LED Row55
- removed sheet LED Row56
- removed sheet LED Row57
- removed sheet LED Row58
- removed sheet LED Row59
- removed sheet LED Row60
- removed sheet LED Row61
- removed sheet LED Row62
- removed sheet LED Row63
- removed sheet LED Row64
- removed sheet LED Row65
- removed sheet LED Row66
- removed sheet LED Row67
- removed sheet LED Row68
- removed sheet LED Row69
- removed sheet LED Row70
- removed sheet LED Row71
- removed sheet LED Row72
- removed sheet LED Row73
- removed sheet LED Row74
- removed sheet LED Row75
- removed sheet LED Row76
- removed sheet LED Row77
- removed sheet LED Row78
- removed sheet LED Row79
- removed sheet LED Row80
- removed sheet LED Row81
- removed sheet LED Row82
- removed sheet LED Row83
- removed sheet LED Row84
- removed sheet LED Row85
- removed sheet LED Row86
- removed sheet LED Row87
- removed sheet LED Row88
- removed sheet LED Row89
- removed sheet LED Row90
- removed sheet LED Row91
- removed sheet LED Row92
- removed sheet LED Row93
- removed sheet LED Row94
- removed sheet LED Row95
- removed sheet LED Row96
- added sheet LED Group (LEDGroup.kicad_sch)
- added sheet LED Group1 (LEDGroup.kicad_sch)
