File: pcb/GrowLight.kicad_pcb (KiCad board)
At the start: 2 copper layers, 190.5 x 81.3 mm, 686 parts, among them J1 Barrel_Jack, Q1 IPT012N08N5, U1 LM555xM

Commit message: fixes
Parts:
- added C1: 100nF, Capacitor_SMD:C_0603_1608Metric, F.Cu at (45.7, 115.2)
- moved H4 217.6 mm to (240.0, 137.5)
- moved FID1 91.6 mm to (234.9, 137.5)
- moved H3 53.6 mm to (240.0, 71.5)
- moved D433 18.3 mm to (49.3, 126.1), turned to 0 degrees
- moved D434 16.0 mm to (49.3, 123.6), turned to 180 degrees
- moved RV1 11.4 mm to (45.9, 122.3)
- moved Q1 10.2 mm to (49.5, 84.2)
- moved FID3 9.92 mm to (52.1, 71.5)
- moved H2 9.56 mm to (47.0, 71.5)
- moved J1 9.51 mm to (50.8, 98.8)
- moved U1 9.16 mm to (47.8, 109.9), turned to -90 degrees
- moved R2 8.87 mm to (49.8, 115.2), turned to -90 degrees
- moved FID2 7.73 mm to (52.1, 137.5)
Routing:
- net (no net): track 24.4 -> 0.00 mm
- net /Control Circuitry/CTRL: track 1.64 -> 24.8 mm, vias 0 -> 2
- net /V_{LED}: track 0.00 -> 22.6 mm, vias 0 -> 2
- net /Control Circuitry/THR: track 0.00 -> 21.8 mm
- net Net-(D433-Pad2): track 0.00 -> 17.8 mm
- net Net-(D434-Pad2): track 0.00 -> 3.15 mm
- net Net-(D433-Pad1): track 0.00 -> 3.12 mm
Other:
- board size 190.5 x 81.3 mm -> 203.2 x 76.2 mm
