File: pcb/GrowLight.kicad_sch (KiCad schematic)
At the start: 9 parts, among them J1 Barrel_Jack_Switch_Pin3Ring, J2 USB_B_Micro, Q1 IPT012N08N5

Commit message: updates
Parts:
- removed J1: Barrel_Jack_Switch_Pin3Ring, Connector_BarrelJack:BarrelJack_GCT_DCJ200-10-A_Horizontal, symbol Connector:Barrel_Jack_Switch_Pin3Ring
- removed J2: USB_B_Micro, Connector_USB:USB_Micro-B_GCT_USB3076-30-A, symbol Connector:USB_B_Micro
- added H4: MountingHole, MountingHole:MountingHole_2.7mm_M2.5_ISO7380, symbol Mechanical:MountingHole
- added J1: Barrel_Jack, Connector_BarrelJack:BarrelJack_GCT_DCJ200-10-A_Horizontal, symbol Connector:Barrel_Jack
Connections:
- net Earth: now also J1.2
- net V_{LED}: now also J1.1
- no-connect marks 1 -> 0
Other:
- removed sheet Voltage Regulator
- sheet Control Circuitry ports: added none; removed V_{DD}, {USB}
- moved on the sheet: FID1, FID2, FID3, H1, H2, H3, Q1
