File: pcb/LEDRow.kicad_sch (KiCad schematic)
At the start: 7 parts

Commit message: updates
Parts:
- R6: value 39 -> 20
Changed lines of the file:
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@@
       (effects (font (size 1.27 1.27)) (justify left))
     )
-    (property "Value" "39" (id 1) (at 97.79 86.3599 0)
+    (property "Value" "20" (id 1) (at 97.79 86.3599 0)
       (effects (font (size 1.27 1.27)) (justify left))
     )

Commit message: fixes
Parts:
- renumbered D7 to D295, D8 to D296, D9 to D297, D10 to D298, D11 to D299, D12 to D300, R6 to R51
Changed lines of the file:
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@@
   (symbol (lib_id "Device:R_US") (at 95.25 85.09 0) (unit 1)
     (in_bom yes) (on_board yes) (fields_autoplaced)
-    (property "Reference" "R6" (id 0) (at 97.79 83.8199 0)
+    (property "Reference" "R51" (id 0) (at 97.79 83.8199 0)
       (effects (font (size 1.27 1.27)) (justify left))
     )
@@
   (symbol (lib_id "Device:LED") (at 95.25 57.15 90) (unit 1)
     (in_bom yes) (on_board yes) (fields_autoplaced)
-    (property "Reference" "D10" (id 0) (at 99.06 57.4674 90)
+    (property "Reference" "D298" (id 0) (at 99.06 57.4674 90)
       (effects (font (size 1.27 1.27)) (justify right))
     )
@@
   (symbol (lib_id "Device:LED") (at 95.25 72.39 90) (unit 1)
     (in_bom yes) (on_board yes) (fields_autoplaced)
-    (property "Reference" "D12" (id 0) (at 99.06 72.7074 90)
+    (property "Reference" "D300" (id 0) (at 99.06 72.7074 90)
       (effects (font (size 1.27 1.27)) (justify right))
     )
@@
   (symbol (lib_id "Device:LED") (at 95.25 49.53 90) (unit 1)
     (in_bom yes) (on_board yes) (fields_autoplaced)
-    (property "Reference" "D9" (id 0) (at 99.06 49.8474 90)
+    (property "Reference" "D297" (id 0) (at 99.06 49.8474 90)
       (effects (font (size 1.27 1.27)) (justify right))
     )
@@
   (symbol (lib_id "Device:LED") (at 95.25 34.29 90) (unit 1)
     (in_bom yes) (on_board yes) (fields_autoplaced)
-    (property "Reference" "D7" (id 0) (at 99.06 34.6074 90)
+    (property "Reference" "D295" (id 0) (at 99.06 34.6074 90)
       (effects (font (size 1.27 1.27)) (justify right))
     )
@@
   (symbol (lib_id "Device:LED") (at 95.25 41.91 90) (unit 1)
     (in_bom yes) (on_board yes) (fields_autoplaced)
-    (property "Reference" "D8" (id 0) (at 99.06 42.2274 90)
+    (property "Reference" "D296" (id 0) (at 99.06 42.2274 90)
       (effects (font (size 1.27 1.27)) (justify right))
     )
@@
   (symbol (lib_id "Device:LED") (at 95.25 64.77 90) (unit 1)
     (in_bom yes) (on_board yes) (fields_autoplaced)
-    (property "Reference" "D11" (id 0) (at 99.06 65.0874 90)
+    (property "Reference" "D299" (id 0) (at 99.06 65.0874 90)
       (effects (font (size 1.27 1.27)) (justify right))
     )
