File: pcb/Control.kicad_sch (KiCad schematic)
At the start: 11 parts, among them IC1 LF2190NTR, SW1 SW_SPST, SW2 SW_SPST, U1 ESP32-C3-MINI-1

Commit message: updates
Parts:
- removed C2: 10uF, Capacitor_SMD:C_1206_3216Metric, symbol Device:C
- removed IC1: LF2190NTR, LF2190:SOIC127P600X175-8N, symbol LF2190NTR:LF2190NTR
- removed R3, R4, R5: 16.9k, Resistor_SMD:R_1206_3216Metric, symbol Device:R_US
- removed SW1, SW2: SW_SPST, Button_Switch_SMD:SW_Push_1P1T_NO_Vertical_Wuerth_434133025816, symbol Switch:SW_SPST
- removed U1: ESP32-C3-MINI-1, Espressif:ESP32-C3-MINI-1, symbol Espressif:ESP32-C3-MINI-1
- added D433: SD0603S040S0R2, Diode_SMD:D_0603_1608Metric, symbol Device:D
- added D434: D, Diode_SMD:D_0603_1608Metric, symbol Device:D
- added U1: LM555xM, Package_SO:SOIC-8_3.9x4.9mm_P1.27mm, symbol Timer:LM555xM
- C1: value 10uF -> 100nF; footprint Capacitor_SMD:C_1206_3216Metric -> (none)
- R2: value 16.9k -> 1k; footprint Resistor_SMD:R_1206_3216Metric -> Resistor_SMD:R_0603_1608Metric
- RV1: footprint Potentiometer_THT:Potentiometer_Alps_RK09Y11_Single_Horizontal -> Potentiometer_THT:Potentiometer_Bourns_PTV09A-2_Single_Horizontal
Connections:
- net CTRL: now also U1.3 (Q)
- net GND: now also C1.2, U1.1 (GND); no longer C1.1, RV1.3
- net V_{CC}: now also R2.1, U1.4 (R), U1.8 (VCC)
- net at R2.2: now also D433.2 (A), D434.1 (K), U1.7 (DIS)
- net THR: now reaches RV1.2
- net THR: now also C1.1, U1.2 (TR), U1.6 (THR)
- removed net V_{DD}: C1.2, R2.1, RV1.1
- new net: D433.1 (K), RV1.3
- new net: D434.2 (A), RV1.1
- no-connect marks 12 -> 1
Other:
- moved on the sheet: RV1

Commit message: fixes
Parts:
- C1: footprint (none) -> Capacitor_SMD:C_0603_1608Metric
Changed lines of the file:
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@@
       (effects (font (size 1.27 1.27)) (justify left))
     )
-    (property "Footprint" "" (id 2) (at 120.3452 77.47 0)
+    (property "Footprint" "Capacitor_SMD:C_0603_1608Metric" (id 2) (at 120.3452 77.47 0)
       (effects (font (size 1.27 1.27)) hide)
     )

Commit message: Updated Diode Name
Parts:
- D434: value D -> SD0603S040S0R2
Changed lines of the file:
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@@
       (effects (font (size 1.27 1.27)) (justify right))
     )
-    (property "Value" "D" (id 1) (at 128.27 55.88 90)
+    (property "Value" "SD0603S040S0R2" (id 1) (at 128.27 55.88 90)
       (effects (font (size 1.27 1.27)) (justify right) hide)
     )
